File: kicad/Display.kicad_sch (KiCad schematic)
At the start: 20 parts, among them J1 FH12A-24S-0.5SH_55_, Q1 BSS138LT1G, SW1 SW_DIP_x02

Commit message: PCB updates (USB to UART circuit)
Connections:
- net VDD_CH343 renamed VDD_UART
Changed lines of the file:
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@@
 		)
 	)
-	(global_label "VDD_CH343"
+	(global_label "VDD_UART"
 		(shape input)
 		(at 102.87 125.73 180)
@@
 		)
 		(property "Intersheetrefs" "${INTERSHEET_REFS}"
-			(at 89.0596 125.73 0)
+			(at 90.6319 125.73 0)
 			(hide yes)
 			(show_name no)
